Commit message: feat: add Schmalz gripper model, flange and tcp frames; fix launch to use our robot description

File: src/fr5_bringup/urdf/fr5_workcell.urdf.xacro (robot description, xacro)
@@ -7,4 +7,13 @@
   <xacro:include filename="$(find fairino_description)/urdf/fairino5_v6.urdf"/>
   <xacro:include filename="$(find fr5_bringup)/urdf/fr5.ros2_control.xacro"/>
+  <xacro:include filename="$(find fr5_bringup)/urdf/schmalz_gripper.xacro"/>
+  <!-- Tool flange face: 100 mm along +z of wrist3_link (FR5 DH d6). -->
+  <joint name="flange_joint" type="fixed">
+    <parent link="wrist3_link"/>
+    <child link="flange"/>
+    <origin xyz="0 0 0.100" rpy="0 0 0"/>
+  </joint>
+  <link name="flange"/>
+  <xacro:schmalz_gripper parent="flange"/>
   <xacro:fr5_ros2_control name="FR5System"
                           use_fake_hardware="$(arg use_fake_hardware)"

Commit message: feat: add D405 wrist mount and camera frame; move gripper onto 9.5 mm mount plate

File: src/fr5_bringup/urdf/fr5_workcell.urdf.xacro (robot description, xacro)
@@ -7,4 +7,5 @@
   <xacro:include filename="$(find fairino_description)/urdf/fairino5_v6.urdf"/>
   <xacro:include filename="$(find fr5_bringup)/urdf/fr5.ros2_control.xacro"/>
+  <xacro:include filename="$(find fr5_bringup)/urdf/d405_wrist_mount.xacro"/>
   <xacro:include filename="$(find fr5_bringup)/urdf/schmalz_gripper.xacro"/>
   <!-- Tool flange face: 100 mm along +z of wrist3_link (FR5 DH d6). -->
@@ -15,5 +16,14 @@
   </joint>
   <link name="flange"/>
-  <xacro:schmalz_gripper parent="flange"/>
+  <!-- Camera mount plate sits on the flange. TODO day 1: set yaw to the arm's real direction. -->
+  <xacro:d405_wrist_mount parent="flange" yaw="0.0"/>
+  <!-- Gripper sits on top of the 9.5 mm mount plate. -->
+  <joint name="tool_adapter_joint" type="fixed">
+    <parent link="flange"/>
+    <child link="tool_adapter"/>
+    <origin xyz="0 0 0.0095" rpy="0 0 0"/>
+  </joint>
+  <link name="tool_adapter"/>
+  <xacro:schmalz_gripper parent="tool_adapter"/>
   <xacro:fr5_ros2_control name="FR5System"
                           use_fake_hardware="$(arg use_fake_hardware)"
