Commit message: Remove obsolete camera post from workcell

File: src/fr5_bringup/urdf/workcell_scene.xacro (robot description, xacro)
@@ -1,5 +1,5 @@
 <?xml version="1.0"?>
 <robot xmlns:xacro="http://www.ros.org/wiki/xacro">
-  <!-- Static workcell from config/workcell.yaml: table, profile, camera post,
+  <!-- Static workcell from config/workcell.yaml: table, profile,
        overhead camera frame and zone frames. Collision shapes keep 1 mm gaps
        so MoveIt never sees permanent contacts. -->
@@ -23,5 +23,4 @@
     <xacro:property name="t" value="${cfg['table']}"/>
     <xacro:property name="p" value="${cfg['profile']}"/>
-    <xacro:property name="c" value="${cfg['camera_post']}"/>
     <xacro:property name="oc" value="${cfg['overhead_camera']}"/>
     <xacro:property name="gap" value="0.001"/>
@@ -57,19 +56,4 @@
       </collision>
     </link>
-    <!-- Wooden camera post: stands on the table (1 mm gap), beside the profile -->
-    <joint name="camera_post_joint" type="fixed">
-      <parent link="base_link"/>
-      <child link="camera_post"/>
-      <origin xyz="${c['center_xy'][0]} ${c['center_xy'][1]} ${t['top_z'] + gap + c['size'][2] / 2}"/>
-    </joint>
-    <link name="camera_post">
-      <visual>
-        <geometry><box size="${c['size'][0]} ${c['size'][1]} ${c['size'][2]}"/></geometry>
-        <material name="wood"><color rgba="0.85 0.72 0.5 1"/></material>
-      </visual>
-      <collision>
-        <geometry><box size="${c['size'][0]} ${c['size'][1]} ${c['size'][2]}"/></geometry>
-      </collision>
-    </link>
     <!-- Overhead camera frame (approximate; replaced by extrinsic calibration) -->
     <joint name="overhead_camera_joint" type="fixed">

Commit message: fix: match measured table and profile heights

File: src/fr5_bringup/urdf/workcell_scene.xacro (robot description, xacro)
@@ -2,6 +2,6 @@
 <robot xmlns:xacro="http://www.ros.org/wiki/xacro">
   <!-- Static workcell from config/workcell.yaml: table, profile,
-       overhead camera frame and zone frames. Collision shapes keep 1 mm gaps
-       so MoveIt never sees permanent contacts. -->
+       overhead camera frame and zone frames. The profile collision box
+       has a 1 mm underside clearance; its physical top surface is preserved. -->
   <!-- Zone frame on the table surface, with a thin visual-only marker -->
   <xacro:macro name="workcell_zone" params="name x y yaw z rgba">
@@ -25,5 +25,5 @@
     <xacro:property name="oc" value="${cfg['overhead_camera']}"/>
     <xacro:property name="gap" value="0.001"/>
-    <xacro:property name="profile_h" value="${-t['top_z'] - 2 * gap}"/>
+    <xacro:property name="profile_h" value="${p['height']}"/>
     <!-- Table top slab: its surface is at top_z -->
     <joint name="table_joint" type="fixed">
@@ -41,9 +41,9 @@
       </collision>
     </link>
-    <!-- Profile: 1 mm below the robot base, 1 mm above the table -->
+    <!-- Physical profile rests on the table; link origin is its centre. -->
     <joint name="profile_joint" type="fixed">
       <parent link="base_link"/>
       <child link="profile"/>
-      <origin xyz="${p['center_xy'][0]} ${p['center_xy'][1]} ${-gap - profile_h / 2}"/>
+      <origin xyz="${p['center_xy'][0]} ${p['center_xy'][1]} ${t['top_z'] + profile_h / 2}"/>
     </joint>
     <link name="profile">
@@ -53,5 +53,7 @@
       </visual>
       <collision>
-        <geometry><box size="${p['size_xy'][0]} ${p['size_xy'][1]} ${profile_h}"/></geometry>
+        <!-- Remove clearance from the underside only. -->
+        <origin xyz="0 0 ${gap / 2}"/>
+        <geometry><box size="${p['size_xy'][0]} ${p['size_xy'][1]} ${profile_h - gap}"/></geometry>
       </collision>
     </link>

Commit message: feat: model measured robot mounting spacer

File: src/fr5_bringup/urdf/workcell_scene.xacro (robot description, xacro)
@@ -24,4 +24,5 @@
     <xacro:property name="p" value="${cfg['profile']}"/>
     <xacro:property name="oc" value="${cfg['overhead_camera']}"/>
+    <xacro:property name="sp" value="${cfg['robot_spacer']}"/>
     <xacro:property name="gap" value="0.001"/>
     <xacro:property name="profile_h" value="${p['height']}"/>
@@ -58,4 +59,26 @@
       </collision>
     </link>
+    <!-- Measured mounting spacer; visual faces meet profile and robot base. -->
+    <joint name="robot_spacer_joint" type="fixed">
+      <parent link="base_link"/>
+      <child link="robot_spacer"/>
+      <origin xyz="${sp['center_xy'][0]} ${sp['center_xy'][1]} ${sp['top_z'] - sp['size'][2] / 2}"/>
+    </joint>
+    <link name="robot_spacer">
+      <visual>
+        <geometry>
+          <box size="${sp['size'][0]} ${sp['size'][1]} ${sp['size'][2]}"/>
+        </geometry>
+        <material name="spacer_aluminium">
+          <color rgba="0.65 0.65 0.68 1"/>
+        </material>
+      </visual>
+      <collision>
+        <!-- Deliberate 1 mm clearance at each fixed mounting face. -->
+        <geometry>
+          <box size="${sp['size'][0]} ${sp['size'][1]} ${sp['size'][2] - 2 * gap}"/>
+        </geometry>
+      </collision>
+    </link>
     <!-- Overhead camera frame (approximate; replaced by extrinsic calibration) -->
     <joint name="overhead_camera_joint" type="fixed">
